Commit message: changes

File: kinect2_bridge/urdf/kinect_v2_standalong_physical.urdf.xacro (robot description, xacro)
@@ -4,6 +4,6 @@
     <link name="root"/>
     <xacro:kinect_v2  parent="root">
-        <origin xyz="2 0 1.04"
-                rpy="0 0 3.141592" /><!-- 2 0 1.04 0 0 3.1415-->
+        <origin xyz="1.8 0 1.04"
+                rpy="0 0 3.141592" /><!-- 1.8 0 1.04 0 0 3.1415-->
     </xacro:kinect_v2>
 </robot>

Commit message: Location of kinect changed

File: kinect2_bridge/urdf/kinect_v2_standalong_physical.urdf.xacro (robot description, xacro)
@@ -4,5 +4,5 @@
     <link name="root"/>
     <xacro:kinect_v2  parent="root">
-        <origin xyz="1.8 0 1.04"
+        <origin xyz="1.65 0 0.965"
                 rpy="0 0 3.141592" /><!-- 1.8 0 1.04 0 0 3.1415-->
     </xacro:kinect_v2>
