Commit message: Update kinect_v2.urdf.xacro

File: kinect2_bridge/urdf/kinect_v2.urdf.xacro (robot description, xacro)
@@ -2,5 +2,5 @@
 <robot name="kinect_v2" xmlns:xacro="http://ros.org/wiki/xacro">
 <xacro:include filename="$(find kinect_v2)/urdf/kinect_v2.gazebo.xacro" />
-    <property name="M_PI" value="3.14159" />
+    <xacro:property name="M_PI" value="3.14159" />
     <!-- Kinect2 and mount assembly -->
     <xacro:macro name="kinect_v2" params=" parent *origin">
